File: K/K.sch (KiCad schematic (older format))
At the start: 1 part

Commit message: hi
Parts:
- removed R?: R, symbol R
- added C? (x8): C, symbol C
- added D? (x2): ESDARF01-1BM2, symbol D_TVS
- added L? (x9): L, symbol L
- added Q?: EPC2038, symbol Q_NMOS_GSD
- added Q? (x2): BFT25A, symbol Q_NPN_BEC
- added Q? (x3): Q_NPN_BEC, symbol Q_NPN_BEC
- added R? (x9): R, symbol R
- added R? (x2): 320, symbol R
- added R? (x4): 50, symbol R
- added U?: TMS320C6748, symbol TMS320C6748
- added U?: BF1105R, symbol BF1105R
Connections:
- net labels added: +3V3, +5V, Aout1, EN1, GND, IN1, MX1, P1
- wire segments 0 -> 47
Other:
- note added: "VG2=1.2V"
