File: K/K.sch (KiCad schematic (older format))
At the start: 42 parts

Commit message: f
Parts:
- removed C?: C, symbol C
- removed L?: L, symbol L
- added C?: C, symbol C
- added D? (x4): MMDL770T1G, symbol D_ALT
- added D? (x6): D_ALT, symbol D_ALT
- added L? (x2): L, symbol L
- added Q?: EPC2038, symbol Q_NMOS_GSD
- added R? (x10): 100, symbol R
- added R? (x10): 10, symbol R
- added R?: 10k, symbol R
Connections:
- net labels added: +12V
- net labels removed: +5V, P1
- wire segments 47 -> 60
Other:
- moved on the sheet: C?, L?, Q?, R?

Commit message: f
Parts:
- removed C? (x5): C, symbol C
- removed D? (x2): ESDARF01-1BM2, symbol D_TVS
- removed L? (x9): L, symbol L
- removed Q? (x3): Q_NPN_BEC, symbol Q_NPN_BEC
- removed R? (x7): R, symbol R
- removed U?: BF1105R, symbol BF1105R
- added L? (x2): L, symbol L
- added R? (x2): 40k, symbol R
- added R? (x2): 1.7k, symbol R
- added R?: 45k, symbol R
- Q?: value BFT25A -> BFU710F
- R?: value R -> 45k
- R?: value R -> 100
Connections:
- net labels removed: +3V3, Aout1, EN1, MX1
- wire segments 60 -> 43
Other:
- note removed: "VG2=1.2V"
- moved on the sheet: C?, L?, Q?, R?
