File: K/_saved_K.sch (KiCad schematic (older format))
At the start: 43 parts

Commit message: f
Parts:
- added D? (x10): D_ALT, symbol D_ALT
- added R? (x10): 100, symbol R
- added R? (x10): 10, symbol R
Connections:
- wire segments 37 -> 57
